File: RoverBaseboard.brd (EAGLE design)
At the start: 87 x 62.9 mm, 57 parts, among them IC3 3.3V, U2 microSD

Commit message: added diode for VUSB/5V so both can be connected safely
Parts:
- added D1: MBR130LSFT1, bt_diode:SOD123FL
Connections:
- new net VUSB: D1.A, U$1.J6-31
- net +5V: now also D1.C
Routing:
- net VUSB: track 0.00 -> 3.38 mm
- net +5V: track 152.4 -> 155.8 mm
Changed lines of the file:
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@@
 <?xml version="1.0" encoding="utf-8"?>
 <!DOCTYPE eagle SYSTEM "eagle.dtd">
-<eagle version="6.4">
+<eagle version="7.1.0">
 <drawing>
 <settings>
@@
 <layer number="21" name="tPlace" color="7" fill="1" visible="no" active="yes"/>
 <layer number="22" name="bPlace" color="7" fill="1" visible="no" active="yes"/>
-<layer number="23" name="tOrigins" color="15" fill="1" visible="no" active="yes"/>
-<layer number="24" name="bOrigins" color="15" fill="1" visible="no" active="yes"/>
-<layer number="25" name="tNames" color="7" fill="1" visible="no" active="yes"/>
-<layer number="26" name="bNames" color="7" fill="1" visible="no" active="yes"/>
+<layer number="23" name="tOrigins" color="15" fill="1" visible="yes" active="yes"/>
+<layer number="24" name="bOrigins" color="15" fill="1" visible="yes" active="yes"/>
+<layer number="25" name="tNames" color="7" fill="1" visible="yes" active="yes"/>
+<layer number="26" name="bNames" color="7" fill="1" visible="yes" active="yes"/>
 <layer number="27" name="tValues" color="7" fill="1" visible="no" active="yes"/>
 <layer number="28" name="bValues" color="7" fill="1" visible="no" active="yes"/>
@@
 <layer number="97" name="Info" color="7" fill="1" visible="no" active="no"/>
 <layer number="98" name="Guide" color="6" fill="1" visible="no" active="no"/>
+<layer number="99" name="SpiceOrder" color="5" fill="1" visible="no" active="no"/>
 <layer number="100" name="Muster" color="7" fill="1" visible="no" active="no"/>
 <layer number="101" name="Hidden" color="15" fill="1" visible="no" active="yes"/>
@@
 <layer number="107" name="Crop" color="7" fill="1" visible="no" active="yes"/>
 <layer number="116" name="Patch_BOT" color="9" fill="4" visible="no" active="yes"/>
-<layer number="121" name="tsilk" color="14" fill="1" visible="yes" active="yes"/>
-<layer number="122" name="bsilk" color="6" fill="1" visible="yes" active="yes"/>
+<layer number="121" name="tsilk" color="14" fill="1" visible="no" active="yes"/>
+<layer number="122" name="bsilk" color="6" fill="1" visible="no" active="yes"/>
 <layer number="125" name="_tNames" color="7" fill="1" visible="no" active="yes"/>
 <layer number="144" name="Drill_legend" color="7" fill="1" visible="no" active="yes"/>
@@
 <pass name="Default">
 <param name="RoutingGrid" value="50mil"/>
+<param name="AutoGrid" value="1"/>
+<param name="Efforts" value="0"/>
+<param name="TopRouterVariant" value="1"/>
 <param name="tpViaShape" value="round"/>
 <param name="PrefDir.1" value="|"/>
@@
 <attribute name="VALUE" x="81.28" y="49.149" size="1.27" layer="27" ratio="10"/>
 </element>
+<element name="D1" library="bt_diode" package="SOD123FL" value="MBR130LSFT1" x="15.24" y="44.45" rot="R270"/>
 </elements>
 <signals>
@@
 <wire x1="10.16" y1="6.35" x2="10.16" y2="12.065" width="0.8128" layer="1"/>
 <wire x1="10.16" y1="12.065" x2="10.287" y2="12.192" width="0.8128" layer="1"/>
+<contactref element="D1" pad="C"/>
+<wire x1="15.24" y1="46.15" x2="15.24" y2="49.53" width="0.8128" layer="1"/>
 </signal>
 <signal name="+3V3">
@@
 <wire x1="58.42" y1="13.97" x2="55.88" y2="16.51" width="0.4064" layer="1"/>
 </signal>
+<signal name="VUSB">
+<contactref element="U$1" pad="J6-31"/>
+<contactref element="D1" pad="A"/>
+<wire x1="15.24" y1="39.37" x2="15.24" y2="42.75" width="0.8128" layer="1"/>
+</signal>
 </signals>
